File: HeadphoneAmp.sch (KiCad schematic (older format))
At the start: 33 parts, among them Q1 IRF540, Q2 IRF540, SW8 SPST, SW9 SPST, U2 ECC82

Commit message: redrawn plus crossfeed, still needs PSU
Parts:
- removed C10: 10uF, symbol CP1
- removed C12: 47uF, symbol CP1
- removed C13, C14: 474, symbol C
- removed C15: 473, symbol C
- removed C16: 1000uF, symbol CP1
- removed GND?, L-OUT?, R-OUT?: CONN_1, symbol CONN_1
- removed IC? (x2): LM317L, v-reg-317L, symbol LM317L
- removed P? (x2): B50K, Pot-POTL_1, symbol POTL_1
- removed Q1: IRF540, TO220, symbol MOSFET_N
- removed R10, R11, R17: 1K, symbol R
- removed R12, R13: 2K2, symbol R
- removed R14: 10R, symbol R
- removed R6: 100K, symbol R
- removed R9: 150R, symbol R
- removed SW8, SW9: SPST, ~, symbol SPST
- removed unit 2 of U2
- added C?: 47uF, symbol CP1
- added C?: 1000uF, symbol CP1
- added C?: 10uF, symbol CP1
- added IC? (x2): LM317TL, v-reg-317TL, symbol LM317TL
- added Q?: IRF510, TO220, symbol MOSFET_N
- added R? (x2): 5K, symbol R
- added R?: 1K, symbol R
- added R?: 10R, symbol R
- added R?: 150R, symbol R
- added R?: 100K, symbol R
- added unit 2 of U1
- added unit 3 of U1
- Q2: value IRF540 -> IRF510
- renumbered U2 to U1
Connections:
- net labels added: L-OUT, R-OUT
- net labels removed: GND
- wire segments 81 -> 50
Other:
- moved on the sheet: C11, C17, C9, Q2, R15, R16, R7, R8, U1A
